Commit message: new commit

File: urdf/turtlebot3_burger.gazebo.xacro (robot description, xacro)
@@ -130,8 +130,8 @@
       <visualize>$(arg camera_visual)</visualize>
       <camera>
-          <horizontal_fov>1.085595</horizontal_fov>
+          <horizontal_fov>1</horizontal_fov>
           <image>
-              <width>800</width>
-              <height>400</height>
+              <width>400</width>
+              <height>300</height>
               <!-- 240 -->
               <format>R8G8B8</format>

File: urdf/turtlebot3_burger.urdf.xacro (robot description, xacro)
@@ -1,4 +1,6 @@
 <?xml version="1.0" ?>
+<!-- model name  -->
 <robot name="turtlebot3_burger_for_autorace" xmlns:xacro="http://ros.org/wiki/xacro">
+  <!-- find model xraco file data  contain comon mesh and robot model gazebo config data  -->
   <xacro:include filename="$(find turtlebot3_autorace_2019)/urdf/common_properties.xacro"/>
   <xacro:include filename="$(find turtlebot3_autorace_2019)/urdf/turtlebot3_burger.gazebo.xacro"/>
@@ -141,7 +143,5 @@
   </link>
   <joint name="camera_joint" type="fixed">
-    <origin xyz="0.040 -0.011 0.10" rpy="0 0.087 0"/>
-    <!-- 8* -->
-    <!-- 0 0.174 0 -->
+    <origin xyz="0.04 0 0.07125" rpy="0  0.3 0"/>
     <parent link="base_link"/>
     <child link="camera_link"/>
@@ -149,13 +149,13 @@
   <link name="camera_link">
     <collision>
-      <origin xyz="0.005 0.011 0.013" rpy="0 0 0"/>
+      <origin xyz="0 0 0" rpy="0 0 0"/>
       <!-- 0.13 -->
       <geometry>
-        <box size="0.015 0.030 0.027"/>
+        <!-- <box size="0.015 0.030 0.027"/> -->
       </geometry>
     </collision>
   </link>
   <joint name="camera_rgb_joint" type="fixed">
-    <origin xyz="0.003 0.011 0.009" rpy="0 0 0"/>
+    <origin xyz="0 0 0" rpy="0 0 0"/>
     <parent link="camera_link"/>
     <child link="camera_rgb_frame"/>
@@ -163,5 +163,5 @@
   <link name="camera_rgb_frame"/>
   <joint name="camera_rgb_optical_joint" type="fixed">
-    <origin xyz="0 0 0" rpy="-1.57 0 -1.57"/>
+    <origin xyz="0 0 0" rpy="0 0 0"/>
     <parent link="camera_rgb_frame"/>
     <child link="camera_rgb_optical_frame"/>
